Commit message: model is more mouse-like

File: mouse_description/urdf/mouse.urdf (robot description, URDF)
Before this commit: robot mouse, 2 links, 1 joints
Links:
- removed link inertia_wheel_roll
- removed link mouse_body
- added link base_link, mass 0.5; collision box size=0.2 0.2 0.2; visual box size=0.4 0.2 0.2
- added link left_back_wheel, mass 1; collision cylinder length=0.05 radius=0.035; visual cylinder length=0.05 radius=0.035
- added link left_front_wheel, mass 1; collision cylinder length=0.05 radius=0.035; visual cylinder length=0.05 radius=0.035
- added link right_back_wheel, mass 1; collision cylinder length=0.05 radius=0.035; visual cylinder length=0.05 radius=0.035
- added link right_front_wheel, mass 1; collision cylinder length=0.05 radius=0.035; visual cylinder length=0.05 radius=0.035
Joints:
- removed joint inertia_wheel_roll_joint
- added joint left_back_wheel_joint: type fixed, parent base_link, child left_back_wheel, origin xyz=-0.133333333333 0.1 -0.135 rpy=0 0 0, axis 0 1 0
- added joint left_front_wheel_joint: type fixed, parent base_link, child left_front_wheel, origin xyz=0.133333333333 0.1 -0.135 rpy=0 0 0, axis 0 1 0
- added joint right_back_wheel_joint: type fixed, parent base_link, child right_back_wheel, origin xyz=-0.133333333333 -0.1 -0.135 rpy=0 0 0, axis 0 1 0
- added joint right_front_wheel_joint: type fixed, parent base_link, child right_front_wheel, origin xyz=0.133333333333 -0.1 -0.135 rpy=0 0 0, axis 0 1 0

Commit message: mouse can now stay without jumping

File: mouse_description/urdf/mouse.urdf (robot description, URDF)
Before this commit: robot mouse, 5 links, 4 joints
Joints:
- joint left_back_wheel_joint: type fixed -> continuous
- joint left_front_wheel_joint: type fixed -> continuous
- joint right_back_wheel_joint: type fixed -> continuous
- joint right_front_wheel_joint: type fixed -> continuous

Commit message: lone mouse walking forward

File: mouse_description/urdf/mouse.urdf (robot description, URDF)
Before this commit: robot mouse, 5 links, 4 joints
Joints:
- joint left_back_wheel_joint: mimic (none) -> joint=left_front_wheel_joint
- joint right_back_wheel_joint: mimic (none) -> joint=right_front_wheel_joint

Commit message: create head for the mouse

File: mouse_description/urdf/mouse.urdf (robot description, URDF)
Before this commit: robot mouse, 5 links, 4 joints
Links:
- added link head, mass 1; collision sphere radius=0.1; visual sphere radius=0.1
Joints:
- added joint neck: type fixed, parent base_link, child head, origin xyz=0.2 0 0 rpy=0 0 0

Commit message: adjust mouse and create arena

File: mouse_description/urdf/mouse.urdf (robot description, URDF)
Before this commit: robot mouse, 6 links, 5 joints
Links:
- link base_link: geometry collision box size=0.4 0.2 0.2; visual box size=0.4 0.2 0.2

Commit message: fix dancing walls and add mouse 3d model

File: mouse_description/urdf/mouse.urdf (robot description, URDF)
Before this commit: robot mouse, 6 links, 5 joints
Links:
- removed link head
- link base_link: geometry collision box size=0.5 0.5 0.5; visual mesh filename=package://mouse_description/meshes/mouse.DAE
Joints:
- removed joint neck

Commit message: fix mouse model and urdf

File: mouse_description/urdf/mouse.urdf (robot description, URDF)
Before this commit: robot mouse, 5 links, 4 joints
Links:
- link base_link: geometry collision box size=0.7 0.5 0.3; visual mesh filename=package://mouse_description/meshes/mouse.DAE
Joints:
- joint left_back_wheel_joint: origin xyz=-0.133333333333 0.1 -0.135 rpy=0 0 0 -> xyz=-0.133333333333 0.1 -0.055 rpy=0 0 0
- joint left_front_wheel_joint: origin xyz=0.133333333333 0.1 -0.135 rpy=0 0 0 -> xyz=0.133333333333 0.1 -0.055 rpy=0 0 0
- joint right_back_wheel_joint: origin xyz=-0.133333333333 -0.1 -0.135 rpy=0 0 0 -> xyz=-0.133333333333 -0.1 -0.055 rpy=0 0 0
- joint right_front_wheel_joint: origin xyz=0.133333333333 -0.1 -0.135 rpy=0 0 0 -> xyz=0.133333333333 -0.1 -0.055 rpy=0 0 0

Commit message: lasers working

File: mouse_description/urdf/mouse.urdf (robot description, URDF)
Before this commit: robot mouse, 5 links, 4 joints
Links:
- added link mouse_sensor; collision cylinder length=0.05 radius=0.035; visual cylinder length=0.05 radius=0.035
Joints:
- added joint sensor_joint: type fixed, parent base_link, child mouse_sensor, origin xyz=0 0 0.5 rpy=0 0 0

Commit message: Fixed mouse spawning for ubuntu 18.04

File: mouse_description/urdf/mouse.urdf (robot description, URDF)
Before this commit: robot mouse, 6 links, 5 joints
Links:
- link base_link: mass 0.5 -> 10; geometry collision box size=0.7 0.5 0.3; visual mesh filename=package://mouse_description/meshes/mouse.dae
- link left_back_wheel: mass 0.25 -> 1
- link left_front_wheel: mass 0.25 -> 1
- link right_back_wheel: mass 0.25 -> 1
- link right_front_wheel: mass 0.25 -> 1

Commit message: Reformulate mouse

File: mouse_description/urdf/mouse.urdf (robot description, URDF)
Before this commit: robot mouse, 6 links, 5 joints
Links:
- removed link left_back_wheel
- removed link left_front_wheel
- removed link right_back_wheel
- removed link right_front_wheel
- added link back_wheel, mass 1; collision sphere radius=0.035; visual sphere radius=0.035
- added link left_wheel, mass 1; collision cylinder length=0.05 radius=0.035; visual cylinder length=0.05 radius=0.035
- added link right_wheel, mass 1; collision cylinder length=0.05 radius=0.035; visual cylinder length=0.05 radius=0.035
Joints:
- removed joint left_back_wheel_joint
- removed joint left_front_wheel_joint
- removed joint right_back_wheel_joint
- removed joint right_front_wheel_joint
- added joint back_wheel_joint: type continuous, parent base_link, child back_wheel, origin xyz=-0.15 0 -0.055 rpy=0 0 0, axis 0 1 0, limit effort=200 velocity=1000.0
- added joint left_wheel_joint: type continuous, parent base_link, child left_wheel, origin xyz=0.133333333333 0.1 -0.055 rpy=0 0 0, axis 0 1 0, limit effort=200 velocity=1000.0
- added joint right_wheel_joint: type continuous, parent base_link, child right_wheel, origin xyz=0.133333333333 -0.1 -0.055 rpy=0 0 0, axis 0 1 0, limit effort=200 velocity=1000.0

Commit message: mouse sensors are working

File: mouse_description/urdf/mouse.urdf (robot description, URDF)
Before this commit: robot mouse, 5 links, 4 joints
Links:
- link mouse_sensor: geometry collision sphere radius=0.01; visual sphere radius=0.01
Joints:
- joint sensor_joint: origin xyz=0 0 0.5 rpy=0 0 0 -> xyz=0.3500001 0 1.1 rpy=0 0 0
