Commit message: Add movement script to launcher

File: mouse_description/urdf/catH.urdf.xacro (robot description, xacro)
@@ -219,10 +219,4 @@
 			<material name="black"/>
 		</visual>
-		<collision>
-			<origin xyz="0 0 0"/>
-			<geometry>
-				<sphere radius="0.01"/>
-			</geometry>
-		</collision>
 	</link>
 	<joint name="sensor_joint" type="fixed">

File: mouse_description/urdf/catK.urdf.xacro (robot description, xacro)
@@ -219,10 +219,4 @@
 			<material name="black"/>
 		</visual>
-		<collision>
-			<origin xyz="0 0 0"/>
-			<geometry>
-				<sphere radius="0.01"/>
-			</geometry>
-		</collision>
 	</link>
 	<joint name="sensor_joint" type="fixed">

File: mouse_description/urdf/mouseA.urdf.xacro (robot description, xacro)
@@ -219,10 +219,4 @@
 			<material name="black"/>
 		</visual>
-		<collision>
-			<origin xyz="0 0 0"/>
-			<geometry>
-				<sphere radius="0.01"/>
-			</geometry>
-		</collision>
 	</link>
 	<joint name="sensor_joint" type="fixed">

File: mouse_description/urdf/mouseO.urdf.xacro (robot description, xacro)
@@ -219,10 +219,4 @@
 			<material name="black"/>
 		</visual>
-		<collision>
-			<origin xyz="0 0 0"/>
-			<geometry>
-				<sphere radius="0.01"/>
-			</geometry>
-		</collision>
 	</link>
 	<joint name="sensor_joint" type="fixed">
