Commit message: Robot can follow walls, run from cats and wander around

File: mouse_description/urdf/mouseA.urdf.xacro (robot description, xacro)
@@ -45,5 +45,5 @@
         <material>Gazebo/FlatBlack</material>
 		<sensor type="ray" name="det_cat_ray_sensor">
-			<pose>0.3500001 0 -0.05 0 0 0</pose>
+			<pose>0.36 0 -0.05 0 0 0</pose>
 			<visualize>true</visualize>
 			<update_rate>40</update_rate>
@@ -229,5 +229,5 @@
 		<parent link="base_link"/>
 		<child link="mouseA_sensor"/>
-		<origin rpy="0 0 0" xyz="0.3500001 0 1.1"/>
+		<origin rpy="0 0 0" xyz="0.36 0 1.1"/>
 	</joint>
 	<gazebo reference="mouseA_sensor">

Commit message: fix wall following vs running from cat

File: mouse_description/urdf/mouseA.urdf.xacro (robot description, xacro)
@@ -44,38 +44,4 @@
         <mu2>1000000.0</mu2>
         <material>Gazebo/FlatBlack</material>
-		<sensor type="ray" name="det_cat_ray_sensor">
-			<pose>0.36 0 -0.05 0 0 0</pose>
-			<visualize>true</visualize>
-			<update_rate>40</update_rate>
-			<ray>
-				<scan>
-					<horizontal>
-						<samples>720</samples>
-						<resolution>1</resolution>
-						<min_angle>-1.9198621772</min_angle>
-						<max_angle>1.9198621772</max_angle>
-					</horizontal>
-				</scan>
-				<range>
-					<min>0.10</min>
-					<max>2.5</max>
-					<resolution>1</resolution>
-				</range>
-				<noise>
-					<type>gaussian</type>
-					<!-- Noise parameters based on published spec for Hokuyo laser
-						achieving "+-30mm" accuracy at range < 10m.  A mean of 0.0m and
-						stddev of 0.01m will put 99.7% of samples within 0.03m of the true
-						reading. -->
-					<mean>0.0</mean>
-					<stddev>0.01</stddev>
-				</noise>
-			</ray>
-			<plugin name="gazebo_ros_mouseA_laser_controller" filename="libgazebo_ros_laser.so">
-				<robotNamespace></robotNamespace>
-				<topicName>/mouseA/laser/cat_scan</topicName>
-				<frameName>mouseA_sensor</frameName>
-			</plugin>
-		</sensor>
     </gazebo>
 	<!-- Right Wheel  -->
@@ -233,5 +199,5 @@
 				<scan>
 					<horizontal>
-						<samples>720</samples>
+						<samples>200</samples>
 						<resolution>1</resolution>
 						<min_angle>-1.9198621772</min_angle>
@@ -261,3 +227,53 @@
 		</sensor>
 	</gazebo>
+	<link name="mouseA_sensor_cat">
+		<visual>
+			<origin xyz="0 0 0"/>
+			<geometry>
+				<sphere radius="0.01"/>
+			</geometry>
+			<material name="black"/>
+		</visual>
+	</link>
+	<joint name="sensor_cat_joint" type="fixed">
+		<parent link="base_link"/>
+		<child link="mouseA_sensor_cat"/>
+		<origin rpy="0 0 0" xyz="0.36 0 -0.05"/>
+	</joint>
+	<gazebo reference="mouseA_sensor_cat">
+		<sensor type="ray" name="det_cat_ray_sensor">
+			<pose>0 0 0 0 0 0</pose>
+			<visualize>true</visualize>
+			<update_rate>40</update_rate>
+			<ray>
+				<scan>
+					<horizontal>
+						<samples>200</samples>
+						<resolution>1</resolution>
+						<min_angle>-1.9198621772</min_angle>
+						<max_angle>1.9198621772</max_angle>
+					</horizontal>
+				</scan>
+				<range>
+					<min>0.10</min>
+					<max>2.5</max>
+					<resolution>1</resolution>
+				</range>
+				<noise>
+					<type>gaussian</type>
+					<!-- Noise parameters based on published spec for Hokuyo laser
+						achieving "+-30mm" accuracy at range < 10m.  A mean of 0.0m and
+						stddev of 0.01m will put 99.7% of samples within 0.03m of the true
+						reading. -->
+					<mean>0.0</mean>
+					<stddev>0.01</stddev>
+				</noise>
+			</ray>
+			<plugin name="gazebo_ros_mouseA_laser_controller" filename="libgazebo_ros_laser.so">
+				<robotNamespace></robotNamespace>
+				<topicName>/mouseA/laser/cat_scan</topicName>
+				<frameName>mouseA_sensor</frameName>
+			</plugin>
+		</sensor>
+	</gazebo>
 </robot>
